Commit message: Camera added to simulation as box

File: src/hsr_support/urdf/xacros/iiwa_14.xacro (robot description, xacro)
@@ -274,16 +274,16 @@
     </joint>
     <link name="${robot_name}_link_ee">
-      <!-- <visual>
-        <origin xyz="0.0 0.0 0.025" rpy="0 0 0"/>
-        <geometry>
-            <box size="0.1 0.05 0.05"/>
-        </geometry>
-      </visual>
-      <collision>
-        <origin xyz="0.0 0.0 0.025" rpy="0 0 0"/>
-        <geometry>
-            <box size="0.1 0.05 0.05"/>
-        </geometry>
-      </collision> -->
+      <visual>
+        <origin xyz="0.0 0.0 0.05" rpy="0 0 0"/>
+        <geometry>
+            <box size="0.1 0.1 0.1"/>
+        </geometry>
+      </visual>
+      <collision>
+        <origin xyz="0.0 0.0 0.05" rpy="0 0 0"/>
+        <geometry>
+            <box size="0.1 0.1 0.1"/>
+        </geometry>
+      </collision>
     </link>
     <!--Extensions -->

Commit message: Sphere trajectory finished

File: src/hsr_support/urdf/xacros/iiwa_14.xacro (robot description, xacro)
@@ -268,20 +268,39 @@
       </collision>
     </link>
+    <joint name="${robot_name}_joint_camera" type="fixed">
+      <parent link="${robot_name}_link_7"/>
+      <child link="${robot_name}_link_camera"/>
+      <origin xyz="0 0 0.126" rpy="0 0 0"/>
+    </joint>
+    <link name="${robot_name}_link_camera">
+      <visual>
+        <origin xyz="0.0 0.0 0.05" rpy="0 0 0"/>
+        <geometry>
+            <box size="0.15 0.1 0.1"/>
+        </geometry>
+      </visual>
+      <collision>
+        <origin xyz="0.0 0.0 0.05" rpy="0 0 0"/>
+        <geometry>
+            <box size="0.15 0.1 0.1"/>
+        </geometry>
+      </collision>
+    </link>
     <joint name="${robot_name}_joint_ee" type="fixed">
-      <parent link="${robot_name}_link_7"/>
+      <parent link="${robot_name}_link_camera"/>
       <child link="${robot_name}_link_ee"/>
-      <origin xyz="0 0 0.126" rpy="0 0 0"/>
+      <origin xyz="0 0 0.10" rpy="0 0 0"/>
     </joint>
     <link name="${robot_name}_link_ee">
       <visual>
-        <origin xyz="0.0 0.0 0.05" rpy="0 0 0"/>
-        <geometry>
-            <box size="0.1 0.1 0.1"/>
-        </geometry>
-      </visual>
-      <collision>
-        <origin xyz="0.0 0.0 0.05" rpy="0 0 0"/>
-        <geometry>
-            <box size="0.1 0.1 0.1"/>
+        <origin xyz="0.0 0.0 0.0" rpy="0 0 0"/>
+        <geometry>
+            <box size="0.0 0.0 0.0"/>
+        </geometry>
+      </visual>
+      <collision>
+        <origin xyz="0.0 0.0 0.0" rpy="0 0 0"/>
+        <geometry>
+            <box size="0.0 0.0 0.0"/>
         </geometry>
       </collision>

Commit message: Mounting plate changed to match reality. Speed increased to maximum

File: src/hsr_support/urdf/xacros/iiwa_14.xacro (robot description, xacro)
@@ -275,13 +275,13 @@
     <link name="${robot_name}_link_camera">
       <visual>
-        <origin xyz="0.0 0.0 0.05" rpy="0 0 0"/>
-        <geometry>
-            <box size="0.15 0.1 0.1"/>
-        </geometry>
-      </visual>
-      <collision>
-        <origin xyz="0.0 0.0 0.05" rpy="0 0 0"/>
-        <geometry>
-            <box size="0.15 0.1 0.1"/>
+        <origin xyz="0.0 0.0 0.025" rpy="0 0 0"/>
+        <geometry>
+            <box size="0.05 0.05 0.05"/>
+        </geometry>
+      </visual>
+      <collision>
+        <origin xyz="0.0 0.0 0.025" rpy="0 0 0"/>
+        <geometry>
+            <box size="0.05 0.05 0.05"/>
         </geometry>
       </collision>
@@ -290,5 +290,5 @@
       <parent link="${robot_name}_link_camera"/>
       <child link="${robot_name}_link_ee"/>
-      <origin xyz="0 0 0.10" rpy="0 0 0"/>
+      <origin xyz="0.00 0.00 0.05" rpy="0 0 0"/>
     </joint>
     <link name="${robot_name}_link_ee">

File: src/hsr_support/urdf/xacros/iiwa_14_mounting_plate.xacro (robot description, xacro)
@@ -6,5 +6,5 @@
       <parent link="${robot_name}_mounting_plate_front_left_bolt"/>
       <child link="${robot_name}_mounting_plate"/>
-      <origin xyz="0.1125 0.1125 0" rpy="0 0 0"/>
+      <origin xyz="0.125 0.125 0" rpy="0 0 0"/>
     </joint>
     <link name="${robot_name}_mounting_plate">
@@ -12,5 +12,5 @@
         <origin xyz="0 0 0.01" rpy="0 0 0"/>
         <geometry>
-          <box size="0.275 0.275 0.02"/>
+          <box size="0.3 0.3 0.02"/>
           <!-- <mesh filename="package://hsr_support/meshes/structure/visual/iiwa_14_mounting_plate.dae"/> -->
         </geometry>
@@ -19,5 +19,5 @@
         <origin xyz="0 0 0.01" rpy="0 0 0"/>
         <geometry>
-          <box size="0.275 0.275 0.02"/>
+          <box size="0.3 0.3 0.02"/>
         </geometry>
       </collision>

Commit message: Add Real camera frame to simulation

File: src/hsr_support/urdf/xacros/iiwa_14.xacro (robot description, xacro)
@@ -2,8 +2,10 @@
 <robot xmlns:xacro="http://www.ros.org/wiki/xacro">
   <!-- some constants -->
-  <xacro:property name="safety_controller_k_pos" value="10" /> <!-- This sets the velocity according the distance the soft limits, velocity = -k_pos * (pos - soft_limit) -->
+  <xacro:property name="safety_controller_k_pos" value="10" />
+  <!-- This sets the velocity according the distance the soft limits, velocity = -k_pos * (pos - soft_limit) -->
   <xacro:property name="safety_controller_k_vel" value="40" />
   <xacro:property name="joint_damping" value="0.0" />
-  <xacro:property name="max_effort" value="300"/> <!-- Should be changed to match the robots specs -->
+  <xacro:property name="max_effort" value="300"/>
+  <!-- Should be changed to match the robots specs -->
   <xacro:property name="PI" value="3.1415926535897931"/>
   <xacro:macro name="iiwa14" params="hardware_interface robot_name">
@@ -16,5 +18,5 @@
         <origin xyz="-0.1 0 0.07" rpy="0 0 0"/>
         <mass value="5"/>
-        <inertia ixx="0.05"  ixy="0"  ixz="0" iyy="0.06" iyz="0" izz="0.03" />
+        <inertia ixx="0.05" ixy="0" ixz="0" iyy="0.06" iyz="0" izz="0.03" />
       </inertial>
       <visual>
@@ -43,10 +45,6 @@
       <origin xyz="0 0 0" rpy="0 0 0" />
       <axis xyz="0 0 1"/>
-      <limit lower="${-169 * PI / 180}" upper="${169 * PI / 180}"
-             effort="${max_effort}" velocity="${85 * PI / 180}" />
-      <safety_controller soft_lower_limit="${-169 * PI / 180}"
-                         soft_upper_limit="${169 * PI / 180}"
-                         k_position="${safety_controller_k_pos}"
-                         k_velocity="${safety_controller_k_vel}"/>
+      <limit lower="${-169 * PI / 180}" upper="${169 * PI / 180}" effort="${max_effort}" velocity="${85 * PI / 180}" />
+      <safety_controller soft_lower_limit="${-169 * PI / 180}" soft_upper_limit="${169 * PI / 180}" k_position="${safety_controller_k_pos}" k_velocity="${safety_controller_k_vel}"/>
       <dynamics damping="${joint_damping}"/>
     </joint>
@@ -55,5 +53,5 @@
         <origin xyz="0 -0.03 0.12" rpy="0 0 0"/>
         <mass value="4"/>
-        <inertia ixx="0.1"  ixy="0"  ixz="0" iyy="0.09" iyz="0" izz="0.02" />
+        <inertia ixx="0.1" ixy="0" ixz="0" iyy="0.09" iyz="0" izz="0.02" />
       </inertial>
       <visual>
@@ -76,10 +74,6 @@
       <origin xyz="-0.00043624 0 0.36" rpy="0 0 0" />
       <axis xyz="0 1 0"/>
-      <limit lower="${-119 * PI / 180}" upper="${119 * PI / 180}"
-             effort="${max_effort}" velocity="${85 * PI / 180}" />
-      <safety_controller soft_lower_limit="${-119 * PI / 180}"
-                         soft_upper_limit="${119 * PI / 180}"
-                         k_position="${safety_controller_k_pos}"
-                         k_velocity="${safety_controller_k_vel}"/>
+      <limit lower="${-119 * PI / 180}" upper="${119 * PI / 180}" effort="${max_effort}" velocity="${85 * PI / 180}" />
+      <safety_controller soft_lower_limit="${-119 * PI / 180}" soft_upper_limit="${119 * PI / 180}" k_position="${safety_controller_k_pos}" k_velocity="${safety_controller_k_vel}"/>
       <dynamics damping="${joint_damping}"/>
     </joint>
@@ -88,5 +82,5 @@
         <origin xyz="0.0003 0.059 0.042" rpy="0 0 0"/>
         <mass value="4"/>
-        <inertia ixx="0.05"  ixy="0"  ixz="0" iyy="0.018" iyz="0" izz="0.044" />
+        <inertia ixx="0.05" ixy="0" ixz="0" iyy="0.018" iyz="0" izz="0.044" />
       </inertial>
       <visual>
@@ -109,10 +103,6 @@
       <origin xyz="0 0 0" rpy="0 0 0" />
       <axis xyz="0 0 1"/>
-      <limit lower="${-169 * PI / 180}" upper="${169 * PI / 180}"
-             effort="${max_effort}" velocity="${100 * PI / 180}" />
-      <safety_controller soft_lower_limit="${-15* PI / 180}"
-                         soft_upper_limit="${15 * PI / 180}"
-                         k_position="${safety_controller_k_pos}"
-                         k_velocity="${safety_controller_k_vel}"/>
+      <limit lower="${-169 * PI / 180}" upper="${169 * PI / 180}" effort="${max_effort}" velocity="${100 * PI / 180}" />
+      <safety_controller soft_lower_limit="${-15* PI / 180}" soft_upper_limit="${15 * PI / 180}" k_position="${safety_controller_k_pos}" k_velocity="${safety_controller_k_vel}"/>
       <dynamics damping="${joint_damping}"/>
     </joint>
@@ -121,5 +111,5 @@
         <origin xyz="0 0.03 0.13" rpy="0 0 0"/>
         <mass value="3"/>
-        <inertia ixx="0.08"  ixy="0"  ixz="0" iyy="0.075" iyz="0" izz="0.01" />
+        <inertia ixx="0.08" ixy="0" ixz="0" iyy="0.075" iyz="0" izz="0.01" />
       </inertial>
       <visual>
@@ -142,10 +132,6 @@
       <origin xyz="0.00043624 0 0.42" rpy="0 0 0" />
       <axis xyz="0 -1 0"/>
-      <limit lower="${-119 * PI / 180}" upper="${119 * PI / 180}"
-             effort="${max_effort}" velocity="${75 * PI / 180}" />
-      <safety_controller soft_lower_limit="${-119 * PI / 180}"
-                         soft_upper_limit="${119 * PI / 180}"
-                         k_position="${safety_controller_k_pos}"
-                         k_velocity="${safety_controller_k_vel}"/>
+      <limit lower="${-119 * PI / 180}" upper="${119 * PI / 180}" effort="${max_effort}" velocity="${75 * PI / 180}" />
+      <safety_controller soft_lower_limit="${-119 * PI / 180}" soft_upper_limit="${119 * PI / 180}" k_position="${safety_controller_k_pos}" k_velocity="${safety_controller_k_vel}"/>
       <dynamics damping="${joint_damping}"/>
     </joint>
@@ -154,5 +140,5 @@
         <origin xyz="0 0.067 0.034" rpy="0 0 0"/>
         <mass value="2.7"/>
-        <inertia ixx="0.03"  ixy="0"  ixz="0" iyy="0.01" iyz="0" izz="0.029" />
+        <inertia ixx="0.03" ixy="0" ixz="0" iyy="0.01" iyz="0" izz="0.029" />
       </inertial>
       <visual>
@@ -175,10 +161,6 @@
       <origin xyz="0 0 0" rpy="0 0 0" />
       <axis xyz="0 0 1"/>
-      <limit lower="${-169 * PI / 180}" upper="${169 * PI / 180}"
-             effort="${max_effort}" velocity="${130 * PI / 180}" />
-      <safety_controller soft_lower_limit="${-169 * PI / 180}"
-                         soft_upper_limit="${169 * PI / 180}"
-                         k_position="${safety_controller_k_pos}"
-                         k_velocity="${safety_controller_k_vel}"/>
+      <limit lower="${-169 * PI / 180}" upper="${169 * PI / 180}" effort="${max_effort}" velocity="${130 * PI / 180}" />
+      <safety_controller soft_lower_limit="${-169 * PI / 180}" soft_upper_limit="${169 * PI / 180}" k_position="${safety_controller_k_pos}" k_velocity="${safety_controller_k_vel}"/>
       <dynamics damping="${joint_damping}"/>
     </joint>
@@ -187,5 +169,5 @@
         <origin xyz="0.0001 0.021 0.076" rpy="0 0 0"/>
         <mass value="1.7"/>
-        <inertia ixx="0.02"  ixy="0"  ixz="0" iyy="0.018" iyz="0" izz="0.005" />
+        <inertia ixx="0.02" ixy="0" ixz="0" iyy="0.018" iyz="0" izz="0.005" />
       </inertial>
       <visual>
@@ -208,10 +190,6 @@
       <origin xyz="0 0 0.4" rpy="0 0 0" />
       <axis xyz="0 1 0"/>
-      <limit lower="${-119 * PI / 180}" upper="${119 * PI / 180}"
-             effort="${max_effort}" velocity="${135 * PI / 180}" />
-      <safety_controller soft_lower_limit="${-119 * PI / 180}"
-                         soft_upper_limit="${119 * PI / 180}"
-                         k_position="${safety_controller_k_pos}"
-                         k_velocity="${safety_controller_k_vel}"/>
+      <limit lower="${-119 * PI / 180}" upper="${119 * PI / 180}" effort="${max_effort}" velocity="${135 * PI / 180}" />
+      <safety_controller soft_lower_limit="${-119 * PI / 180}" soft_upper_limit="${119 * PI / 180}" k_position="${safety_controller_k_pos}" k_velocity="${safety_controller_k_vel}"/>
       <dynamics damping="${joint_damping}"/>
     </joint>
@@ -220,5 +198,5 @@
         <origin xyz="0 0.0006 0.0004" rpy="0 0 0"/>
         <mass value="1.8"/>
-        <inertia ixx="0.005"  ixy="0"  ixz="0" iyy="0.0036" iyz="0" izz="0.0047" />
+        <inertia ixx="0.005" ixy="0" ixz="0" iyy="0.0036" iyz="0" izz="0.0047" />
       </inertial>
       <visual>
@@ -239,12 +217,9 @@
       <parent link="${robot_name}_link_6"/>
       <child link="${robot_name}_link_7"/>
-      <origin xyz="0 0 0" rpy="0 0 0"/>3BS
-      <axis xyz="0 0 1"/>
-      <limit lower="${-174 * PI / 180}" upper="${174 * PI / 180}"
-             effort="${max_effort}" velocity="${135 * PI / 180}" />
-      <safety_controller soft_lower_limit="${-172 * PI / 180}"
-                         soft_upper_limit="${172 * PI / 180}"
-                         k_position="${safety_controller_k_pos}"
-                         k_velocity="${safety_controller_k_vel}"/>
+      <origin xyz="0 0 0" rpy="0 0 0"/>
+3BS
+      <axis xyz="0 0 1"/>
+      <limit lower="${-174 * PI / 180}" upper="${174 * PI / 180}" effort="${max_effort}" velocity="${135 * PI / 180}" />
+      <safety_controller soft_lower_limit="${-172 * PI / 180}" soft_upper_limit="${172 * PI / 180}" k_position="${safety_controller_k_pos}" k_velocity="${safety_controller_k_vel}"/>
       <dynamics damping="${joint_damping}"/>
     </joint>
@@ -253,5 +228,5 @@
         <origin xyz="0 0 0.02" rpy="0 0 0"/>
         <mass value="0.3"/>
-        <inertia ixx="0.001"  ixy="0"  ixz="0" iyy="0.001" iyz="0" izz="0.001" />
+        <inertia ixx="0.001" ixy="0" ixz="0" iyy="0.001" iyz="0" izz="0.001" />
       </inertial>
       <visual>
@@ -275,13 +250,13 @@
     <link name="${robot_name}_link_camera">
       <visual>
-        <origin xyz="0.0 0.0 0.025" rpy="0 0 0"/>
-        <geometry>
-            <box size="0.05 0.05 0.05"/>
-        </geometry>
-      </visual>
-      <collision>
-        <origin xyz="0.0 0.0 0.025" rpy="0 0 0"/>
-        <geometry>
-            <box size="0.05 0.05 0.05"/>
+        <origin xyz="0.0 0.0 0.00" rpy="0 0 0"/>
+        <geometry>
+          <mesh filename="package://hsr_support/meshes/iiwa_14/visual/D405_mount.dae"/>
+        </geometry>
+      </visual>
+      <collision>
+        <origin xyz="0.0 0.0 0.00" rpy="0 0 0"/>
+        <geometry>
+          <mesh filename="package://hsr_support/meshes/iiwa_14/collision/D405_mount.stl"/>
         </geometry>
       </collision>
@@ -290,5 +265,5 @@
       <parent link="${robot_name}_link_camera"/>
       <child link="${robot_name}_link_ee"/>
-      <origin xyz="0.00 0.00 0.05" rpy="0 0 0"/>
+      <origin xyz="-0.010 0.00 0.05" rpy="0 0 0"/>
     </joint>
     <link name="${robot_name}_link_ee">
@@ -296,5 +271,5 @@
         <origin xyz="0.0 0.0 0.0" rpy="0 0 0"/>
         <geometry>
-            <box size="0.0 0.0 0.0"/>
+          <box size="0.0 0.0 0.0"/>
         </geometry>
       </visual>
@@ -302,17 +277,14 @@
         <origin xyz="0.0 0.0 0.0" rpy="0 0 0"/>
         <geometry>
-            <box size="0.0 0.0 0.0"/>
+          <box size="0.0 0.0 0.0"/>
         </geometry>
       </collision>
     </link>
     <!--Extensions -->
-    <xacro:if value="$(arg use_ros2_control)" >
+    <xacro:if value="$(arg use_ros2_control)">
       <xacro:include filename="$(find hsr_support)/urdf/xacros/control/iiwa.ros2_control.xacro" />
-      <xacro:iiwa_position_only name="IiwaPositionHardwareInterface"
-                                robot_ip="$(arg robot_ip)"
-                                robot_port="$(arg robot_port)"
-                                hardware="$(arg hardware)"/>
+      <xacro:iiwa_position_only name="IiwaPositionHardwareInterface" robot_ip="$(arg robot_ip)" robot_port="$(arg robot_port)" hardware="$(arg hardware)"/>
     </xacro:if>
-    <xacro:unless value="$(arg use_ros2_control)" >
+    <xacro:unless value="$(arg use_ros2_control)">
       <xacro:include filename="$(find hsr_support)/urdf/xacros/iiwa.transmission.xacro" />
       <xacro:iiwa_transmission hardware_interface="${hardware_interface}" robot_name="${robot_name}"/>
