Commit message: Pointclouds from all points of motion

File: src/hsr_support/urdf/xacros/d405.xacro (robot description, xacro)
@@ -68,5 +68,5 @@
             <mesh filename="package://hsr_support/meshes/d405/d405.dae" />
           </geometry>
-          <material name="aluminum"/>
+          <material name="aluminium"/>
         </xacro:if>
         <xacro:unless value="${use_mesh}">

File: src/hsr_support/urdf/xacros/iiwa_14.xacro (robot description, xacro)
@@ -246,5 +246,5 @@
       <parent link="${robot_name}_link_7"/>
       <child link="${robot_name}_link_camera"/>
-      <origin xyz="0 0 0.126" rpy="0 0 0"/>
+      <origin xyz="0 0 0.126" rpy="0 0 ${pi}"/>
     </joint>
     <link name="${robot_name}_link_camera">
