Commit message: Apply CBH optical table as collision box
Change optical table offset from z = 0.006 to 0.0 and rotation to 0, to work in positive quadrant

File: src/hsr_support/urdf/iiwa_workcell.urdf.xacro (robot description, xacro)
@@ -10,5 +10,6 @@
         <parent link="world"/>
         <child link="optical_table"/>
-        <origin xyz="0.0 0.0 0.006" rpy="0.0 0.0 ${pi/2}"/>
+        <origin xyz="0.0 0.0 0.0" rpy="0.0 0.0 0.0"/>
+        <!-- Change offset from z = 0.006 to 0.0 and rotation to 0, to work in positive quadrant -->
     </joint>
     <xacro:optical_table />

File: src/hsr_support/urdf/xacros/optical_table.xacro (robot description, xacro)
@@ -4,13 +4,17 @@
     <link name="optical_table">
       <visual>
-        <origin xyz="0 0 0" rpy="0 0 0"/>
+        <origin xyz="0.45 0.375 0.03" rpy="0 0 0"/>
+        <geometry>
+            <box size="0.9 0.75 0.06"/>
+        </geometry>
+        <!-- <origin xyz="0 0 0" rpy="0 0 0"/>
         <geometry>
           <mesh filename="package://hsr_support/meshes/structure/visual/B90120A.dae"/>
-        </geometry>
+        </geometry> -->
       </visual>
       <collision>
-        <origin xyz="0.6 0.45 0.03" rpy="0 0 0"/>
+        <origin xyz="0.45 0.375 0.03" rpy="0 0 0"/>
         <geometry>
-            <box size="1.2 0.9 0.06"/>
+            <box size="0.9 0.75 0.06"/>
         </geometry>
       </collision>
@@ -29,15 +33,15 @@
       <parent link="optical_table"/>
       <child link="optical_table_back_left_bolt"/>
-      <origin xyz="0.0125 0.8875 0.06" rpy="0 0 0"/>
+      <origin xyz="0.0125 0.7375 0.06" rpy="0 0 0"/>
     </joint>
     <joint name="optical_table_front_right_bolt_joint" type="fixed">
       <parent link="optical_table"/>
       <child link="optical_table_front_right_bolt"/>
-      <origin xyz="1.1875 0.0125 0.06" rpy="0 0 0"/>
+      <origin xyz="0.8875 0.0125 0.06" rpy="0 0 0"/>
     </joint>
     <joint name="optical_table_back_right_bolt_joint" type="fixed">
       <parent link="optical_table"/>
       <child link="optical_table_back_right_bolt"/>
-      <origin xyz="1.1875 0.8875 0.06" rpy="0 0 0"/>
+      <origin xyz="0.8875 0.7375 0.06" rpy="0 0 0"/>
     </joint>
   </xacro:macro>

Commit message: Swap XY to match CBH table

File: src/hsr_support/urdf/iiwa_workcell.urdf.xacro (robot description, xacro)
@@ -17,5 +17,5 @@
         <parent link="optical_table_front_left_bolt"/>
         <child link="$(arg iiwa_name)_mounting_plate_front_left_bolt"/>
-        <origin xyz="0.025 0.025 0.00" rpy="0.0 0.0 0"/>
+        <origin xyz="0.025 0.025 0.00" rpy="0.0 0.0 0.0"/>
     </joint>
     <xacro:iiwa_14_mounting_plate robot_name="$(arg iiwa_name)"/>
@@ -23,6 +23,7 @@
         <parent link="$(arg iiwa_name)_mounting_plate_centre_top_surface"/>
         <child link="$(arg iiwa_name)_link_0"/>
-        <origin xyz="0 0 0" rpy="0.0 0.0 ${pi}"/>
+        <origin xyz="0 0 0" rpy="0.0 0.0 ${pi/2} "/>
     </joint>
+    <!-- ${pi} -->
     <xacro:iiwa14 hardware_interface="$(arg hardware_interface)" robot_name="$(arg iiwa_name)">
     </xacro:iiwa14>

File: src/hsr_support/urdf/xacros/optical_table.xacro (robot description, xacro)
@@ -4,7 +4,7 @@
     <link name="optical_table">
       <visual>
-        <origin xyz="0.45 0.375 0.03" rpy="0 0 0"/>
+        <origin xyz="0.375 0.45 0.03" rpy="0 0 0"/>
         <geometry>
-            <box size="0.9 0.75 0.06"/>
+            <box size="0.75 0.9 0.06"/>
         </geometry>
         <!-- <origin xyz="0 0 0" rpy="0 0 0"/>
@@ -14,7 +14,7 @@
       </visual>
       <collision>
-        <origin xyz="0.45 0.375 0.03" rpy="0 0 0"/>
+        <origin xyz="0.375 0.45 0.03" rpy="0 0 0"/>
         <geometry>
-            <box size="0.9 0.75 0.06"/>
+            <box size="0.75 0.9 0.06"/>
         </geometry>
       </collision>
@@ -33,15 +33,15 @@
       <parent link="optical_table"/>
       <child link="optical_table_back_left_bolt"/>
-      <origin xyz="0.0125 0.7375 0.06" rpy="0 0 0"/>
+      <origin xyz="0.7375 0.0125 0.06" rpy="0 0 0"/>
     </joint>
     <joint name="optical_table_front_right_bolt_joint" type="fixed">
       <parent link="optical_table"/>
       <child link="optical_table_front_right_bolt"/>
-      <origin xyz="0.8875 0.0125 0.06" rpy="0 0 0"/>
+      <origin xyz="0.0125 0.8875 0.06" rpy="0 0 0"/>
     </joint>
     <joint name="optical_table_back_right_bolt_joint" type="fixed">
       <parent link="optical_table"/>
       <child link="optical_table_back_right_bolt"/>
-      <origin xyz="0.8875 0.7375 0.06" rpy="0 0 0"/>
+      <origin xyz="0.7375 0.8875 0.06" rpy="0 0 0"/>
     </joint>
   </xacro:macro>

Commit message: Update iiwa xacros

File: src/hsr_support/urdf/iiwa_workcell.urdf.xacro (robot description, xacro)
@@ -11,5 +11,4 @@
         <child link="optical_table"/>
         <origin xyz="0.0 0.0 0.0" rpy="0.0 0.0 0.0"/>
-        <!-- Change offset from z = 0.006 to 0.0 and rotation to 0, to work in positive quadrant -->
     </joint>
     <xacro:optical_table />
@@ -25,13 +24,24 @@
         <origin xyz="0 0 0" rpy="0.0 0.0 ${pi/2} "/>
     </joint>
-    <!-- ${pi} -->
     <xacro:iiwa14 hardware_interface="$(arg hardware_interface)" robot_name="$(arg iiwa_name)">
     </xacro:iiwa14>
-    <!-- <link name="(arg iiwa_name)_camera_frame"></link>
-    <joint name="$(arg iiwa_name)_camera_joint" type="fixed">
+    <!-- <joint name="$(arg iiwa_name)_camera_joint" type="fixed">
         <parent link="$(arg iiwa_name)_link_ee"/>
         <child link="$(arg iiwa_name)_camera_frame"/>
-        <origin xyz="0 0 0.05" rpy="0.0 0.0 0"/>
+        <origin xyz="0 0 0.0" rpy="0.0 0.0 0"/>
     </joint>
-     -->
+    <link name="(arg iiwa_name)_camera_frame">
+        <visual>
+            <origin xyz="0.0 0.0 0.025" rpy="0 0 0"/>
+            <geometry>
+                <box size="0.1 0.05 0.05"/>
+            </geometry>
+        </visual>
+        <collision>
+            <origin xyz="0.0 0.0 0.025" rpy="0 0 0"/>
+            <geometry>
+                <box size="0.1 0.05 0.05"/>
+            </geometry>
+        </collision>
+    </link> -->
 </robot>

File: src/hsr_support/urdf/xacros/iiwa_14.xacro (robot description, xacro)
@@ -274,4 +274,16 @@
     </joint>
     <link name="${robot_name}_link_ee">
+      <!-- <visual>
+        <origin xyz="0.0 0.0 0.025" rpy="0 0 0"/>
+        <geometry>
+            <box size="0.1 0.05 0.05"/>
+        </geometry>
+      </visual>
+      <collision>
+        <origin xyz="0.0 0.0 0.025" rpy="0 0 0"/>
+        <geometry>
+            <box size="0.1 0.05 0.05"/>
+        </geometry>
+      </collision> -->
     </link>
     <!--Extensions -->

Commit message: Add camera urdf srdf and desccription

File: src/hsr_support/urdf/iiwa_workcell.urdf.xacro (robot description, xacro)
@@ -4,4 +4,5 @@
     <xacro:include filename="$(find hsr_support)/urdf/xacros/iiwa_14.xacro"/>
     <xacro:include filename="$(find hsr_support)/urdf/xacros/optical_table.xacro"/>
+    <xacro:include filename="$(find hsr_support)/urdf/xacros/d405.xacro"/>
     <xacro:include filename="$(find hsr_support)/urdf/xacros/iiwa_14_mounting_plate.xacro"/>
     <xacro:arg name="iiwa_name" default="iiwa"/>
@@ -24,24 +25,8 @@
         <origin xyz="0 0 0" rpy="0.0 0.0 ${pi/2} "/>
     </joint>
+    <xacro:d405 parent="$(arg iiwa_name)_link_camera">
+        <origin xyz="0 -0.021 0.04535" rpy="0.0 ${-pi/2} ${-pi/2} "/>
+    </xacro:d405>
     <xacro:iiwa14 hardware_interface="$(arg hardware_interface)" robot_name="$(arg iiwa_name)">
     </xacro:iiwa14>
-    <!-- <joint name="$(arg iiwa_name)_camera_joint" type="fixed">
-        <parent link="$(arg iiwa_name)_link_ee"/>
-        <child link="$(arg iiwa_name)_camera_frame"/>
-        <origin xyz="0 0 0.0" rpy="0.0 0.0 0"/>
-    </joint>
-    <link name="(arg iiwa_name)_camera_frame">
-        <visual>
-            <origin xyz="0.0 0.0 0.025" rpy="0 0 0"/>
-            <geometry>
-                <box size="0.1 0.05 0.05"/>
-            </geometry>
-        </visual>
-        <collision>
-            <origin xyz="0.0 0.0 0.025" rpy="0 0 0"/>
-            <geometry>
-                <box size="0.1 0.05 0.05"/>
-            </geometry>
-        </collision>
-    </link> -->
 </robot>

File: src/hsr_support/urdf/xacros/iiwa_14.xacro (robot description, xacro)
@@ -265,5 +265,5 @@
       <parent link="${robot_name}_link_camera"/>
       <child link="${robot_name}_link_ee"/>
-      <origin xyz="-0.010 0.00 0.05" rpy="0 0 0"/>
+      <origin xyz="-0.010 0.00 0.06" rpy="0 0 0"/>
     </joint>
     <link name="${robot_name}_link_ee">
